File: franzininho-rev1.sch (KiCad schematic (older format))
At the start: 17 parts, among them J1 CONN_01X08, SW1 SW_RESET, U1 ATTINY85-20PU, U2 USB_conn

Commit message: add board layout
Parts:
- U2: footprint usb_copper:USB_COPPER -> usb_copper:USB_COPPER_2
Changed lines of the file:
@@
 F 0 "U2" H 3250 3625 60  0000 C CNN
 F 1 "USB_conn" H 3250 4225 60  0000 C CNN
-F 2 "usb_copper:USB_COPPER" H 3250 3925 60  0001 C CNN
+F 2 "usb_copper:USB_COPPER_2" H 3250 3925 60  0001 C CNN
 F 3 "" H 3250 3925 60  0001 C CNN
 	1    3250 3925
